File: eagle/oresat-minusz-end-card.sch (EAGLE design)
At the start: 17 parts, among them J1 J-SAMTEC-TFM-110-X1-XXX-D-RA, J2 U.FL, J3 U.FL, J4 U.FL

Commit message: Updated end cards with antenna keep outs, and rewired +Z end card debug port and started on +Z schematic update with power domain.
Parts:
- removed CM4, CM5, CM6, CM7: ORESAT-SOLARPANEL-CARD-12PIN, oresat-connectors:ORESAT-SOLARPANEL-CARD-12PIN
- added C1: 10u, oresat-rcl:C-EU0603-B-NOSILK
- added C10, C11: 22u, oresat-rcl:C-EU0805-B-NOSILK
- added C12, C15, C18, C2, C8: 100n, rcl_custom:C-EU0402-B-NOSILK
- added C13, C14: 20p, rcl_custom:C-EU0402-B-NOSILK
- added C3, C7: 10u, oresat-rcl:C-EU0805-B-NOSILK
- added C9: 22u, oresat-rcl:C-EU0603-B-NOSILK
- added CF1: M55-7011242R, J-Harwin-M55-6021242R:J-HARWIN-M55-6021242R
- added D1: GREEN, SparkFun-LED:LED-GREEN0603
- added J5, J6: M55-7101242R, J-Harwin-M55-7101242:M55-7101242R
- added J7, J9: U.FL, SparkFun-Connectors:U.FL2PIN
- added J8: FTSH-105-XX-X-DV-K, J-Samtec-FTSH-105-XXX-DV-K-ARM-SWD:FTSH-105-XX-X-DV-K
- added L1: 1.5 uH, L-Coilcraft-XFL4020:L-COILCRAFT-XFL4020
- added R1, R11, R4, R8: 10k, rcl_custom:R-US_0402-B-NOSILK
- added R10, R7: 4.7k, rcl_custom:R-US_0402-B-NOSILK
- added R2: 470k, rcl_custom:R-US_0402-B-NOSILK
- added R3: 150k, rcl_custom:R-US_0402-B-NOSILK
- added R5, R6: NP, rcl_custom:R-US_0402-B-NOSILK
- added R9: 2.7k, rcl_custom:R-US_0402-B-NOSILK
- added TP1, TP2, TP3, TP4: TPPAD1-13, testpad:TPPAD1-13
- added TP11, TP12, TP13, TP14, TP15, TP7: TEST-POINT, Tova:TEST-POINT
- added U2: TPS63070, ic-pwr-tps63070x:TPS63070X
- added U3: TCAN330, TCAN330:TCAN330
- added U4: STM32F042K6, STM32F042K:STM32F042K6
- added X2: 16MHZ-2.5x2mm, low-gain-radio:CRYSTAL-WITH-GND
- J3, J4: value U.FL -> M55-7101242R; device SparkFun-Connectors:U.FL2PIN -> J-Harwin-M55-7101242:M55-7101242R
Connections:
- net AUX_CAN2_H renamed CAN2_H
- net AUX_CAN2_L renamed CAN2_L
- removed net AUX_!SHUTDOWN: J1.19, J1.20, JP9.10
- removed net AUX_CAN1_H: J1.13, J1.14, JP9.7
- removed net AUX_CAN1_L: J1.15, J1.16, JP9.8
- removed net AUX_GND1: J1.17, J1.18, JP9.9
- removed net AUX_GND2: J1.11, J1.12, JP9.6
- removed net AUX_GND3: J1.10, J1.9, JP9.5
- removed net AUX_VBUS1: J1.7, J1.8, JP9.4
- removed net AUX_VBUS2: J1.5, J1.6, JP9.3
- removed net N$300: CM3.CENTER, J4.SIGNAL
- new net !SHUTDOWN: J1.19, J1.20, J3.1, J3.2, J4.1, J4.2, J5.1, J5.2, J6.1, J6.2, JP9.10
- new net 3.3V: C10.1, C11.1, C12.2, C15.2, C18.2, C8.2, C9.1, CF1.11, CF1.12, J8.VTREF, R10.2, R11.2, R2.2, R5.2, R7.2, TP11.1, U2.VOUT, U3.VCC, U4.VDD, U4.VDDA, U4.VDDIO2
- new net BOOT1: R8.2, TP7.1, U4.PB8-BOOT0
- new net CAN1_H: J1.13, J1.14, J3.10, J3.9, J4.10, J4.9, J5.10, J5.9, J6.10, J6.9, JP9.7, U3.CANH
- new net CAN1_L: J1.15, J1.16, J3.11, J3.12, J4.11, J4.12, J5.11, J5.12, J6.11, J6.12, JP9.8, U3.CANL
- new net CAN_RX: U3.RXD, U4.PA11
- new net CAN_SHDN: U3.SHDN, U4.PA10
- new net CAN_SILENT: U3.S, U4.PA9
- new net CAN_TX: U3.TXD, U4.PA12
- new net CRYSTALIN1: C14.1, U4.PF0-OSC_IN, X2.1
- new net CRYSTALOUT1: C13.1, U4.PF1-OSC_OUT, X2.2
- new net N$1: J4.7, J4.8, TP2.TP
- new net N$2: J3.7, J3.8, TP1.TP
- new net N$4: J5.7, J5.8, TP3.TP
- new net N$5: J6.7, J6.8, TP4.TP
- new net N$7: D1.A, R9.1
- new net NRESET: J8.!RESET, U4.NRST
- new net PA0: R9.2, U4.PA0
- new net PA1: U4.PA1
- new net PA15: U4.PA15
- new net PA2/USART2_TX: U4.PA2
- new net PA3/USART2_RX: U4.PA3
- new net PA4: U4.PA4
- new net PA5/SPI1_SCK: U4.PA5
- new net PA6/SPI1_MISO: U4.PA6
- new net PA7/SPI1_MOSI: U4.PA7
- new net PA8: U4.PA8
- new net PB0: U4.PB0
- new net PB1: U4.PB1
- new net PB3: U4.PB3
- new net PB4/I2C-!RESET: CF1.3, CF1.4, U4.PB4
- new net PB5/I2C-!INT: CF1.5, CF1.6, R11.1, U4.PB5
- new net PB6/SCL: CF1.7, CF1.8, R7.1, U4.PB6
- new net PB7/SDA: CF1.10, CF1.9, R10.1, U4.PB7
- new net RF3: CM3.CENTER, J9.SIGNAL
- new net SWCLK: J8.SWDCLK/TCK, U4.PA14-SWCLK
- new net SWDIO: J8.SWDIO/TMS, U4.PA13-SWDIO
- new net TPS-EN2: R1.1, R6.2, TP15.1, U2.EN, U2.PS/SYNC
- new net TPS-FB2: R2.1, R3.2, U2.FB
- new net TPS-FB4: TP13.1, U2.FB2
- new net TPS-L1: L1.1, U2.L1
- new net TPS-L2: L1.2, U2.L2
- new net TPS-PG2: R5.1, TP12.1, U2.PG
- new net TPS-VAUX2: C2.1, U2.VAUX
- new net TPS-VSEL2: R4.2, TP14.1, U2.VSEL
- new net VBUS: C1.1, C3.1, C7.1, J1.5, J1.6, J1.7, J1.8, J3.5, J3.6, J4.5, J4.6, J5.5, J5.6, J6.5, J6.6, JP9.3, JP9.4, R1.2, U2.VIN
- net GND: now also C1.2, C10.2, C11.2, C12.1, C13.2, C14.2, C15.1, C18.1, C2.2, C3.2, C7.2, C8.1, C9.2, CF1.1, CF1.2, CF1.SHIELDS, D1.C, J1.10, J1.11, J1.12, J1.17, J1.18, J1.9, J3.3, J3.4, J3.SHIELD, J4.3, J4.4, J4.SHIELD, J5.3, J5.4, J5.SHIELD, J6.3, J6.4, J6.SHIELD, J7.GND, J8.GND, J8.GND@2, J8.GNDDET, J9.GND, JP9.5, JP9.6, JP9.9, R3.1, R4.1, R6.1, R8.1, U2.GND, U2.PGND, U3.GND, U4.VSS, X2.SHIELD; no longer J3.GND, J4.GND
- net RF2: now also J7.SIGNAL; no longer J3.SIGNAL
Other:
- note added: "!RESET to the TCA should be pulled high by the STM"
- note added: "+X+Z Solar panel"
- note added: "+Y+Z Solar panel"
- note added: "-X+Z Solar panel"
- note added: "-Y+Z Solar panel"
- note added: "0603"
- note added: "0805"
- note added: "10 pn 1.27mm ARM SWD connector"
- note added: "CAN Transceiver"
- note added: "Debug Connector"
- note added: "End Cap Connector"
- note added: "NRST pull-up built in"
- moved on the sheet: CM1, CM2, CM3, J2, JP9
