File: eagle/oresat-plusz-end-card.sch (EAGLE design)
At the start: 54 parts, among them J2 U.FL, J3 M55-7101242R, J4 M55-7101242R, J5 M55-7101242R, J6 M55-7101242R, J7 J-SAMTEC-TFM-120-X1-XXX-D-RA, J8 FTSH-105-XX-X-DV-K, U2 TPS63070, U3 TCAN330, U4 STM32F042K6, X2 16MHZ-2.5x2mm

Commit message: Added OreSat power domain -- via design blocksgit status -- and OMG it's doneish.
Parts:
- removed C1: 10u, oresat-rcl:C-EU0603-B-NOSILK
- removed C10: 22u, oresat-rcl:C-EU0805-B-NOSILK
- removed C2: 100n, rcl_custom:C-EU0402-B-NOSILK
- removed C3, C7: 10u, oresat-rcl:C-EU0805-B-NOSILK
- removed R1, R4: 10k, rcl_custom:R-US_0402-B-NOSILK
- removed R2: 470k, rcl_custom:R-US_0402-B-NOSILK
- removed R3: 150k, rcl_custom:R-US_0402-B-NOSILK
- removed R5, R6: NP, rcl_custom:R-US_0402-B-NOSILK
- removed TP11, TP12, TP13, TP14, TP15: TEST-POINT, Tova:TEST-POINT
- removed U2: TPS63070, ic-pwr-tps63070x:TPS63070X
- added C16, C19, C20: 1u, oresat-rcl:C-EU0603-B-NOSILK
- added C17: 22u, oresat-rcl:C-EU0805-B-NOSILK
- added C6: 100n, rcl_custom:C-EU0402-B-NOSILK
- added D5, D6: GREEN, SparkFun-LED:LED-GREEN0603
- added D7: AMBER, SparkFun-LED:LED-GREEN0603
- added Q1, Q2: MOSFET-PCH-SOT23-6, Q-MOSFET-PCH-SOT23-6:MOSFET-PCH-SOT23-6
- added Q7, Q8: PMV45EN, Tova:PMV45EN
- added R39, R40, R71: 2.7k, rcl_custom:R-US_0402-B-NOSILK
- added R41, R54, R55: 100, rcl_custom:R-US_0402-B-NOSILK
- added R42, R43, R44, R45, R46, R47, R48, R49, R50, R51, R52, R53, R62, R64, R66, R67, R70: NP, rcl_custom:R-US_0402-B-NOSILK
- added R56, R57, R58, R60, R65, R68, R69: 10k, rcl_custom:R-US_0402-B-NOSILK
- added R59: 100m, rcl:R-US_R1206
- added R61, R63: 0, rcl_custom:R-US_0402-B-NOSILK
- added TP24, TP25, TP26, TP27, TP28, TP29, TP30, TP31, TP32, TP33, TP34, TP35, TP36, TP37, TP38, TP39, TP40, TP41: TEST-POINT, Tova:TEST-POINT
- added U10: MCP1703A, v-reg:XC63FPM
- added U6: MAX7310ATE, U-Maxim-MAX7310-I2C-GPIO-expander:MAX7310
- added U8: MAX4211CETE, U-Maxim-MAX4211-power-monitor:MAX4211
- added U9: TPS62111RSA, U-TI-TPS6211x-SPS-buck:TPS6211X
- C11: value 22u -> 10u
- C9: value 22u -> NP; device oresat-rcl:C-EU0603-B-NOSILK -> rcl_custom:C-EU0402-B-NOSILK
- L1: value 1.5 uH -> 6.8u; device L-Coilcraft-XFL4020:L-COILCRAFT-XFL4020 -> L-ECS-MPI4040:L-ECS-MPI4040; DIS Mouser -> (none); DPN 994-XFL4020-152MEB -> (none); MFR Coilcraft -> ECS; MPN XFL4020-152ME -> ECS-MPI4040R4-6R8-R
Connections:
- removed net TPS-EN2: R1.1, R6.2, TP15.1, U2.EN, U2.PS/SYNC
- removed net TPS-FB2: R2.1, R3.2, U2.FB
- removed net TPS-FB4: TP13.1, U2.FB2
- removed net TPS-L1: L1.1, U2.L1
- removed net TPS-L2: L1.2, U2.L2
- removed net TPS-PG2: R5.1, TP12.1, U2.PG
- removed net TPS-VAUX2: C2.1, U2.VAUX
- removed net TPS-VSEL2: R4.2, TP14.1, U2.VSEL
- new net !FAULT: Q8.D, R68.1, TP29.1, U6.IO2
- new net AD0: R42.1, R43.2, R44.2, R45.1, U6.AD0
- new net AD1: R46.1, R47.2, R48.2, R49.1, U6.AD1
- new net AD2: R50.1, R51.2, R52.2, R53.1, U6.AD2
- new net CB-RESET: R60.2, TP28.1, U6.IO1, U8.CIN2-
- new net CB_CTRL: Q1.G, Q8.G, R65.1, U8.COUT1, U8.COUT2, U8.LE
- new net MAX4211-3V3: C20.1, U10.OUT, U8.VCC
- new net N$10: Q2.G, Q7.D, R57.1
- new net N$11: Q2.D, R59.1, U8.RS+
- new net N$12: R61.1, R62.2, TP26.1, U8.CIN1-
- new net N$13: R63.1, R64.2, TP25.1, U8.CIN1+
- new net N$14: R61.2, U8.IOUT
- new net N$16: R63.2, U8.CIN2+, U8.REF
- new net N$17: TP24.1, U8.POUT
- new net N$18: R67.1, U8.INHIBIT
- new net N$19: C9.1, R66.2, R67.2
- new net N$20: C19.1, Q1.S, R59.2, R65.2, U10.IN, U8.RS-
- new net N$21: TP35.1, U6.IO3
- new net N$22: TP36.1, U6.IO4
- new net N$23: TP37.1, U6.IO5
- new net N$24: TP38.1, U6.IO6
- new net N$25: R71.2, TP39.1, U6.IO7
- new net N$26: D7.A, R71.1
- new net N$6: D5.A, R39.1
- new net N$8: D6.A, R40.1
- new net N$9: R56.1, U6.!RESET
- new net ON/!OFF: Q7.G, R58.2, TP27.1, U6.IO0
- new net PEN-SCL-FILT: R43.1, R47.1, R51.1, R54.2, TP40.1, U6.SCL
- new net PEN-SDA-FILT: R45.2, R49.2, R53.2, R55.2, TP41.1, U6.SDA
- new net TPS62111-PG1: TP31.1, U9.PG
- new net TPS62111-SYNC1: R69.1, R70.2, TP32.1, U9.SYNC
- new net TPS62111_SW1: L1.1, U9.SW
- new net VBUSP: C11.1, C16.1, C9.2, Q1.D, R39.2, R69.2, TP30.1, U9.EN, U9.VIN
- new net VPD: C6.2, R41.2, R42.2, R46.2, R50.2, R56.2, R68.2, TP34.1, U6.V+
- net 3.3V: now also C17.1, L1.2, R40.2, TP33.1, U9.FB; no longer C10.1, C11.1, C9.1, R2.2, R5.2, TP11.1, U2.VOUT
- net GND: now also C16.2, C17.2, C19.2, C20.2, C6.1, D5.C, D6.C, D7.C, Q7.S, Q8.S, R44.1, R48.1, R52.1, R58.1, R60.1, R62.1, R64.1, R66.1, R70.1, U10.GND, U6.GND, U8.GND, U9.GND, U9.LBI, U9.LBO; no longer C1.2, C10.2, C2.2, C3.2, C7.2, C9.2, R3.1, R4.1, R6.1, U2.GND, U2.PGND
- net OPD_PWR: now also R41.1
- net OPD_SCL: now also R54.1
- net OPD_SDA: now also R55.1
- net VBUS: now also Q2.S, R57.2; no longer C1.1, C3.1, C7.1, R1.2, U2.VIN
Other:
- note added: "(3.3V)"
- note added: "3.1"
- note added: "3.3V Card Switching Supply"
- note added: "Address selection for Card (See MAX7310 datasheet)"
- note added: "Card Power Switch and Circuit Breaker"
- note added: "ECS-MPI4040R4-6R8-R"
- note added: "Main Power Switch"
- note added: "OreSat Power Domain (OPD) Controller"
- note added: "OreSat Power Domain (OPD) Power Supply (3.3V)"
- note added: "OreSat Power Enable (PEN)"
- note added: "Vbus = (6.0,7.2,8.4)V"
