File: oresat-minusz-end-card/oresat-minusz-end-card.kicad_sch (KiCad schematic)
At the start: 59 parts

Commit message: Fixed some errors on the ancient -z end card
Parts:
- C1, C9: footprint (none) -> oresat-minusz-end-card:.0603-B-NOSILK
- C10, C11: value (none) -> 22u; footprint (none) -> oresat-minusz-end-card:.0805-B-NOSILK
- C12, C13, C14, C15, C18, C2, C8, R1, R10, R11, R2, R3, R4, R5, R6, R7, R8, R9: footprint (none) -> oresat-minusz-end-card:.0402-B-NOSILK
- C3, C7: value (none) -> 10u; footprint (none) -> oresat-minusz-end-card:.0805-B-NOSILK
- CF1: value (none) -> M55-7011242R; footprint (none) -> oresat-minusz-end-card:HARWIN-M55-6021242R
- CM1, CM2, CM3: value (none) -> J-MOLEX-SMPM-73300-003X; footprint (none) -> oresat-footprints:J-MOLEX-SMPM-073300-003X; symbol oresat-minusz-end-card-eagle-import:J-MOLEX-SMPM-73300-003X -> OreSat-j-molex-smpm-73300-003x:J-MOLEX-SMPM-73300-003X
- D1: value (none) -> GREEN; footprint (none) -> oresat-minusz-end-card:LED-0603
- H1, H2, H3, H4: value (none) -> STAND-OFFTIGHT; footprint (none) -> oresat-minusz-end-card:STAND-OFF-TIGHT
- J1: footprint (none) -> oresat-minusz-end-card:J-SAMTEC-TFM-110-X1-XXX-D-RA
- J2, J7, J9: value (none) -> U.FL; footprint (none) -> oresat-footprints:J-U.FL; symbol oresat-minusz-end-card-eagle-import:U.FL2PIN -> OreSat-u.fl2pin:U.FL2PIN
- J3, J4, J5, J6: value (none) -> M55-7101242R; footprint (none) -> oresat-minusz-end-card:M55-7101242R
- J8: footprint (none) -> oresat-minusz-end-card:CON10_2X5_DUK_FTSH
- JP9: value (none) -> PINHD-1X10; footprint (none) -> oresat-minusz-end-card:1X10
- L1: footprint (none) -> oresat-minusz-end-card:L-COILCRAFT-XFL4020
- TP1, TP2, TP3, TP4: value (none) -> TPPAD1-13; footprint (none) -> oresat-minusz-end-card:P1-13
- TP11, TP12, TP13, TP14, TP15, TP7: value (none) -> TEST-POINT; footprint (none) -> oresat-minusz-end-card:2MM-TEST-POINT
- U2: footprint (none) -> oresat-minusz-end-card:TPS63070X
- U3: footprint (none) -> oresat-minusz-end-card:SOT23-8_TI-DCN
- U4: footprint (none) -> oresat-minusz-end-card:QFP32-7X7
- X2: footprint (none) -> oresat-minusz-end-card:CRYSTAL_2.5X2
Connections:
- net GND: now also CM1.GND (SHIELD3), CM2.GND (SHIELD3), CM3.GND (SHIELD3), J2.GND, J7.GND, J9.GND; no longer CM1.P$1 (SHIELD3), CM1.P$2 (SHIELD2), CM1.P$3 (SHIELD1), CM1.P$4 (SHIELD), CM2.P$1 (SHIELD3), CM2.P$2 (SHIELD2), CM2.P$3 (SHIELD1), CM2.P$4 (SHIELD), CM3.P$1 (SHIELD3), CM3.P$2 (SHIELD2), CM3.P$3 (SHIELD1), CM3.P$4 (SHIELD), J2.1 (GND), J2.2 (GND), J7.1 (GND), J7.2 (GND), J9.1 (GND), J9.2 (GND)
Other:
- note added: "Connectors"
- note added: "Power"
- note added: "STM32"
- note removed: "2.0"
- moved on the sheet: C1, C10, C11, C12, C13, C14, C15, C18, C2, C3, C7, C8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
