File: dev-boards/BalUn-eval-board/balun-eval-board.kicad_pcb (KiCad board)
At the start: 4 copper layers, 7 parts, among them J2 Conn_Coaxial_142-0711-201, J3 Conn_Coaxial_142-0711-201, J4 Conn_Coaxial_142-0711-201, U1 NCS2-62+

Commit message: made changes to BalUn board
Parts:
- moved J4 104.2 mm to (159.2, 75.5), turned to 90 degrees
- moved C1 89.3 mm to (139.6, 76.2), turned to 90 degrees
- moved TP1 83.8 mm to (135.8, 49.3)
- moved TP2 72.6 mm to (135.8, 100.5)
- moved U1 66.6 mm to (136.7, 74.9)
- moved J3 55.0 mm to (124.3, 85.5), turned to 90 degrees
- moved J2 49.5 mm to (124.3, 64.3)
Routing:
- net Net-(J2-Pad3): track 0.00 -> 36.0 mm
- net Net-(C1-Pad2): track 0.00 -> 21.6 mm
- net Net-(J3-Pad3): track 20.6 -> 36.0 mm
- added copper zone on B.Cu, net GND
- added copper zone on F.Cu, net GND
