File: dev-boards/BalUn-eval-board/balun-eval-board.kicad_pcb (KiCad board)
At the start: 4 copper layers, 7 parts, among them J2 Conn_Coaxial_142-0711-201, J3 Conn_Coaxial_142-0711-201, J4 Conn_Coaxial_142-0711-201, U1 NCS2-62+

Commit message: BalUn board v2
Parts:
- removed J4: Conn_Coaxial_142-0711-201, oresat-connectors:SMA 142-0711-201
- added J1: SMA-142-0711-821, oresat-connectors:SMA-142-0711-821, F.Cu at (101.2, 94.8)
- added R1: 0, oresat-passives:0603-B-NOSILK, F.Cu at (121.6, 112.8)
- added R2: 0, oresat-passives:0603-B-NOSILK, F.Cu at (121.6, 91.0)
- added R3: 0, oresat-passives:0603-B-NOSILK, F.Cu at (117.8, 94.8)
- added R4: 0, oresat-passives:0603-B-NOSILK, F.Cu at (117.8, 109.0)
- J2, J3: value Conn_Coaxial_142-0711-201 -> SMA-142-0711-821; footprint oresat-connectors:SMA 142-0711-201 -> oresat-connectors:SMA-142-0711-821
- moved J2 50.3 mm to (101.2, 109.0)
- moved TP1 32.0 mm to (121.6, 78.0)
- moved J3 31.7 mm to (151.0, 102.6), turned to -90 degrees
- moved C1 30.4 mm to (125.7, 103.3)
- moved U1 30.4 mm to (122.8, 101.9)
- moved TP2 29.1 mm to (121.6, 125.8)
Connections:
- J2 pad 1: GND -> Net-(J2-Pad1)
- J2 pad 3: Net-(J2-Pad3) -> GND
- J3 pad 1: GND -> Net-(C1-Pad2)
- J3 pad 3: Net-(J3-Pad3) -> GND
- TP1 pad 1: Net-(J2-Pad3) -> Net-(R2-Pad1)
- TP2 pad 1: Net-(J3-Pad3) -> Net-(R1-Pad2)
- U1 pad 1: Net-(J2-Pad3) -> Net-(R2-Pad2)
- U1 pad 3: Net-(J3-Pad3) -> Net-(R1-Pad1)
Routing:
- net Net-(J3-Pad3): track 36.0 -> 0.00 mm
- net Net-(J2-Pad3): track 36.0 -> 0.00 mm
- net Net-(R1-Pad2): track 0.00 -> 12.3 mm
- net Net-(R2-Pad1): track 0.00 -> 12.2 mm
- net Net-(R2-Pad2): track 0.00 -> 12.1 mm
- net Net-(R1-Pad1): track 0.00 -> 12.1 mm
- net Net-(J2-Pad1): track 0.00 -> 10.8 mm
- net Net-(J1-Pad1): track 0.00 -> 10.8 mm
- net Net-(C1-Pad2): track 21.6 -> 22.4 mm
- net GND: vias 46 -> 0
Other:
- board outline added: 44.5 x 55.8 mm
