File: dev-boards/BalUn-eval-board/balun-eval-board.kicad_sch (KiCad schematic)
At the start: 7 parts, among them J2 Conn_Coaxial_142-0711-201, J3 Conn_Coaxial_142-0711-201, J4 Conn_Coaxial_142-0711-201, U1 NCS2-62+

Commit message: BalUn board v2
Parts:
- removed J2, J3, J4: Conn_Coaxial_142-0711-201, oresat-connectors:SMA 142-0711-201, symbol oresat-symbols:Conn_Coaxial_142-0711-201
- added J1, J2, J3: SMA-142-0711-821, oresat-connectors:SMA-142-0711-821, symbol oresat-connectors:SMA-142-0711-821
- added R1, R2, R3, R4: 0, oresat-passives:0603-B-NOSILK, symbol Device:R
Connections:
- net GND: now also J1.2 (In), J1.3 (Ext), J1.4 (Ext), J1.5 (Ext), J2.2 (In), J2.3 (Ext), J2.4 (Ext), J2.5 (Ext), J3.2 (In), J3.3 (Ext), J3.4 (Ext), J3.5 (Ext)
- net at C1.2, U1.4: now also J3.1
- net at TP2.1: now also R1.2; no longer U1.3
- net at U1.1: now also R2.2, R3.1; no longer TP1.1
- new net: J1.1, R3.2
- new net: R2.1, TP1.1
- new net: R1.1, R4.1, U1.3
- new net: J2.1, R4.2
Other:
- moved on the sheet: TP1, TP2

Commit message: made changes to BalUn board
Parts:
- removed J1, J2, J3: SMA-142-0711-821, oresat-connectors:SMA-142-0711-821, symbol oresat-connectors:SMA-142-0711-821
- removed R1, R2, R3, R4: 0, oresat-passives:0603-B-NOSILK, symbol Device:R
- added J1, J2, J3: SMA-142-0711-201, oresat-connectors:SMA-J-P-H-ST-EM1, symbol oresat-connectors:SMA-J-P-H-ST-EM1
Connections:
- net GND: now also J1.2 (In), J1.3 (Ext), J2.2 (In), J2.3 (Ext), J3.2 (In), J3.3 (Ext)
- net at U1.1: now also TP1.1, J1.1
- net at C1.2, U1.4: now also J3.1
- net at TP2.1: now also U1.3, J2.1

Commit message: made changes to NCS2-62+ balUn dev board
Changed lines of the file:
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@@
-	)
-	(junction
-		(at 69.85 90.17)
-		(diameter 0)
-		(color 0 0 0 0)
-	)
-	(junction
-		(at 93.98 104.14)
-		(diameter 0)
-		(color 0 0 0 0)
 	)
 	(junction
@@
 	(wire
 		(pts
-			(xy 69.85 90.17) (xy 68.58 90.17)
+			(xy 109.22 90.17) (xy 124.46 90.17)
 		)
 		(stroke
@@
 	(wire
 		(pts
-			(xy 109.22 90.17) (xy 124.46 90.17)
+			(xy 102.87 100.33) (xy 109.22 100.33)
 		)
 		(stroke
@@
 	(wire
 		(pts
-			(xy 102.87 100.33) (xy 109.22 100.33)
+			(xy 109.22 100.33) (xy 124.46 100.33)
 		)
 		(stroke
@@
 	(wire
 		(pts
-			(xy 109.22 100.33) (xy 124.46 100.33)
+			(xy 82.55 90.17) (xy 90.17 90.17)
 		)
 		(stroke
@@
 	(wire
 		(pts
-			(xy 82.55 90.17) (xy 90.17 90.17)
+			(xy 109.22 77.47) (xy 109.22 90.17)
 		)
 		(stroke
@@
 	(wire
 		(pts
-			(xy 109.22 77.47) (xy 109.22 90.17)
+			(xy 109.22 100.33) (xy 109.22 114.3)
 		)
 		(stroke
@@
 	(wire
 		(pts
-			(xy 109.22 100.33) (xy 109.22 114.3)
+			(xy 102.87 90.17) (xy 109.22 90.17)
 		)
 		(stroke
@@
 	(wire
 		(pts
-			(xy 102.87 90.17) (xy 109.22 90.17)
+			(xy 68.58 90.17) (xy 82.55 90.17)
 		)
 		(stroke
@@
 		)
 	)
-	(wire
-		(pts
-			(xy 82.55 90.17) (xy 69.85 90.17)
-		)
-		(stroke
-			(width 0)
-			(type default)
-		)
-	)
 	(symbol
 		(lib_id "Device:C")
@@
 	)
 	(symbol
-		(lib_id "power:PWR_FLAG")
-		(at 69.85 90.17 0)
-		(mirror y)
-		(unit 1)
-		(body_style 1)
-		(exclude_from_sim no)
-		(in_bom yes)
-		(on_board yes)
-		(in_pos_files yes)
-		(dnp no)
-		(fields_autoplaced yes)
-		(property "Reference" "#FLG01"
-			(at 69.85 86.614 0)
-			(hide yes)
-			(show_name no)
-			(do_not_autoplace no)
-			(effects
-				(font
-					(size 1.27 1.27)
-				)
-			)
-		)
-		(property "Value" "PWR_FLAG"
-			(at 69.85 85.09 0)
-			(hide yes)
-			(show_name no)
-			(do_not_autoplace no)
-			(effects
-				(font
-					(size 1.27 1.27)
-				)
-			)
-		)
-		(property "Footprint" ""
-			(at 69.85 90.17 0)
-			(hide yes)
-			(show_name no)
-			(do_not_autoplace no)
-			(effects
-				(font
-					(size 1.27 1.27)
-				)
-			)
-		)
-		(property "Datasheet" ""
-			(at 69.85 90.17 0)
-			(hide yes)
-			(show_name no)
-			(do_not_autoplace no)
-			(effects
-				(font
-					(size 1.27 1.27)
-				)
-			)
-		)
-		(property "Description" "Special symbol for telling ERC where power comes from"
-			(at 69.85 90.17 0)
-			(hide yes)
-			(show_name no)
-			(do_not_autoplace no)
-			(effects
-				(font
-					(size 1.27 1.27)
-				)
-			)
-		)
-		(pin "1"
-		)
-		(instances
-			(project "balun-eval-board"
-				(path "/8436592f-ebd9-43cb-82bb-370e94da9621"
-					(reference "#FLG01")
-					(unit 1)
-				)
-			)
-		)
-	)
-	(symbol
 		(lib_id "oresat-symbols:GND")
 		(at 93.98 104.14 0)
@@
 					(unit 1)
 				)
-			)
-		)
-	)
-	(symbol
-		(lib_name "PWR_FLAG_1")
-		(lib_id "power:PWR_FLAG")
-		(at 93.98 104.14 90)
-		(mirror x)
-		(unit 1)
-		(body_style 1)
-		(exclude_from_sim no)
-		(in_bom yes)
-		(on_board yes)
-		(in_pos_files yes)
-		(dnp no)
-		(fields_autoplaced yes)
-		(property "Reference" "#FLG02"
-			(at 92.075 104.14 0)
-			(hide yes)
-			(show_name no)
-			(do_not_autoplace no)
-			(effects
-				(font
-					(size 1.27 1.27)
-				)
-			)
-		)
-		(property "Value" "PWR_FLAG"
-			(at 90.17 104.1399 90)
-			(hide yes)
-			(show_name no)
-			(do_not_autoplace no)
-			(effects
-				(font
-					(size 1.27 1.27)
-				)
-				(justify left)
-			)
-		)
-		(property "Footprint" ""
-			(at 93.98 104.14 0)
-			(hide yes)
-			(show_name no)
-			(do_not_autoplace no)
-			(effects
-				(font
-					(size 1.27 1.27)
-				)
-			)
-		)
-		(property "Datasheet" ""
-			(at 93.98 104.14 0)
-			(hide yes)
-			(show_name no)
-			(do_not_autoplace no)
-			(effects
-				(font
-					(size 1.27 1.27)
-				)
-			)
-		)
-		(property "Description" "Special symbol for telling ERC where power comes from"
-			(at 93.98 104.14 0)
-			(hide yes)
-			(show_name no)
-			(do_not_autoplace no)
-			(effects
-				(font
-					(size 1.27 1.27)
-				)
-			)
-		)
-		(pin "1"
-		)
-		(instances
-			(project "balun-eval-board"
-				(path "/8436592f-ebd9-43cb-82bb-370e94da9621"
-					(reference "#FLG02")
-					(unit 1)
-				)
