File: oresat1-minusz-end-card/oresat1-minusz-end-card.kicad_sch (KiCad schematic)
At the start: 31 parts, among them J1 J-SAMTEC-TFM-120-01-L-D-RA, J2 U.FL-R-SMT-1, J3 M55-7101242R, J5 M55-7101242R

Commit message: Changes to minus Z
Resolved 2 git issues. Added led test light to deployer circuit to test deployment
Parts:
- J4, J6: value ~ -> (none)
Connections:
- no-connect marks 19 -> 20

Commit message: Routine push
Parts:
- J1: renamed from CM1; value 2477330-1 -> 733000020
- J2: renamed from CM2; value 2477330-1 -> 733000020
- J3: renamed from CM3; value 2477330-1 -> 733000020
Connections:
- net GND: now also J1.2 (SHLD), J2.2 (SHLD), J3.2 (SHLD); no longer J1.SHLD, J2.SHLD, J3.SHLD
- net L1BAND: now also J1.1 (SIG); no longer J1.SIG
- net LBAND: now also J2.1 (SIG); no longer J2.SIG
- net UHF: now also J3.1 (SIG); no longer J3.SIG
- no-connect marks 20 -> 16
Other:
- sheet OPD ports: added none; removed MY-UART-RX, MY-UART-TX, PY-UART-RX, PY-UART-TX
- note removed: "+Y SM is DNP"
- note removed: "-Y SM is DNP"
Changed lines of the file:
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@@
 		)
 	)
-	(text "+Y SM is DNP"
-		(exclude_from_sim no)
-		(at 182.88 63.754 0)
-		(effects
-			(font
-				(size 1.27 1.27)
-				(thickness 0.1588)
-			)
-		)
-	)
 	(text "To L band monopole"
 		(exclude_from_sim no)
@@
 		)
 	)
-	(text "-Y SM is DNP"
-		(exclude_from_sim no)
-		(at 182.626 78.74 0)
-		(effects
-			(font
-				(size 1.27 1.27)
-				(thickness 0.1588)
-			)
-		)
-	)
 	(text "L Band Feed System (1.265 GHz)"
 		(exclude_from_sim no)
@@
 	)
 	(no_connect
-		(at 173.99 77.47)
-	)
-	(no_connect
 		(at 73.66 80.01)
 	)
@@
 	)
 	(no_connect
-		(at 173.99 62.23)
-	)
-	(no_connect
 		(at 73.66 107.95)
 	)
@@
 	)
 	(no_connect
-		(at 173.99 64.77)
-	)
-	(no_connect
 		(at 73.66 52.07)
 	)
@@
 	)
 	(no_connect
-		(at 173.99 80.01)
-	)
-	(no_connect
 		(at 73.66 44.45)
 	)
@@
 	(wire
 		(pts
-			(xy 172.72 80.01) (xy 173.99 80.01)
-		)
-		(stroke
-			(width 0)
-			(type default)
-		)
-	)
-	(wire
-		(pts
 			(xy 229.87 161.29) (xy 224.79 161.29)
 		)
@@
 	(wire
 		(pts
-			(xy 172.72 64.77) (xy 173.99 64.77)
-		)
-		(stroke
-			(width 0)
-			(type default)
-		)
-	)
-	(wire
-		(pts
 			(xy 203.2 166.37) (xy 229.87 166.37)
 		)
@@
 	(wire
 		(pts
-			(xy 172.72 77.47) (xy 173.99 77.47)
-		)
-		(stroke
-			(width 0)
-			(type default)
-		)
-	)
-	(wire
-		(pts
 			(xy 203.2 57.15) (xy 172.72 57.15)
 		)
@@
 	(wire
 		(pts
-			(xy 172.72 62.23) (xy 173.99 62.23)
-		)
-		(stroke
-			(width 0)
-			(type default)
-		)
-	)
-	(wire
-		(pts
 			(xy 73.66 39.37) (xy 82.55 39.37)
 		)
@@
 		(in_pos_files yes)
 		(dnp no)
-		(property "Reference" "CM3"
+		(property "Reference" "J3"
 			(at 74.93 220.98 0)
 			(show_name no)
@@
 			)
 		)
-		(property "Value" "2477330-1"
+		(property "Value" "733000020"
 			(at 74.93 223.52 0)
 			(show_name no)
@@
 			)
 		)
-		(property "Datasheet" "https://www.te.com/commerce/DocumentDelivery/DDEController?Action=srchrtrv&DocNm=SMPM_Connectors_Product_Extension-en&DocType=Data+Sheet&DocLang=English&DocFormat=pdf&PartCntxt=2477330-1"
+		(property "Datasheet" "https://tools.molex.com/pdm_docs/sd/733000020_sd.pdf"
 			(at 69.85 208.28 0)
 			(hide yes)
@@
 			)
 		)
-		(property "Description" "SMPM Connector Plug, Male Pin 50 Ohms Board Edge, Cutout; Surface Mount Solder"
+		(property "Description" "SMPM Connector Plug, Male Pin 50Ohm Board Edge, Cutout; Surface Mount Solder"
 			(at 69.85 217.17 0)
 			(hide yes)
@@
 			)
 		)
-		(pin "SHLD"
+		(pin "2"
 		)
-		(pin "SIG"
+		(pin "1"
 		)
 		(instances
 			(project "oresat1-minusz-end-card"
 				(path "/f7595184-4323-4ed9-b19e-5e32e3c6e76f"
-					(reference "CM3")
+					(reference "J3")
 					(unit 1)
 				)
@@
 	)
 	(symbol
+		(lib_name "J-MOLEX-SMPM-73300-002X_1")
 		(lib_id "oresat-connectors:J-MOLEX-SMPM-73300-002X")
 		(at 68.58 154.94 0)
@@
 		(in_pos_files yes)
 		(dnp no)
-		(property "Reference" "CM1"
+		(property "Reference" "J1"
 			(at 73.66 158.75 0)
 			(show_name no)
@@
 			)
 		)
-		(property "Value" "2477330-1"
+		(property "Value" "733000020"
 			(at 73.66 161.29 0)
 			(show_name no)
@@
 			)
 		)
-		(property "Datasheet" "https://www.te.com/commerce/DocumentDelivery/DDEController?Action=srchrtrv&DocNm=SMPM_Connectors_Product_Extension-en&DocType=Data+Sheet&DocLang=English&DocFormat=pdf&PartCntxt=2477330-1"
+		(property "Datasheet" "https://tools.molex.com/pdm_docs/sd/733000020_sd.pdf"
 			(at 68.58 146.05 0)
 			(hide yes)
@@
 			)
 		)
-		(property "Description" "SMPM Connector Plug, Male Pin 50 Ohms Board Edge, Cutout; Surface Mount Solder"
+		(property "Description" "SMPM Connector Plug, Male Pin 50Ohm Board Edge, Cutout; Surface Mount Solder"
 			(at 68.58 154.94 0)
 			(hide yes)
@@
 			)
 		)
-		(pin "SHLD"
+		(pin "2"
 		)
-		(pin "SIG"
+		(pin "1"
 		)
 		(instances
 			(project "oresat1-minusz-end-card"
 				(path "/f7595184-4323-4ed9-b19e-5e32e3c6e76f"
-					(reference "CM1")
+					(reference "J1")
 					(unit 1)
 				)
@@
 	)
 	(symbol
+		(lib_name "J-MOLEX-SMPM-73300-002X_2")
 		(lib_id "oresat-connectors:J-MOLEX-SMPM-73300-002X")
 		(at 68.58 185.42 0)
@@
 		(in_pos_files yes)
 		(dnp no)
-		(property "Reference" "CM2"
+		(property "Reference" "J2"
 			(at 73.66 189.23 0)
 			(show_name no)
@@
 			)
 		)
-		(property "Value" "2477330-1"
+		(property "Value" "733000020"
 			(at 73.66 191.77 0)
 			(show_name no)
@@
 			)
 		)
-		(property "Datasheet" "https://www.te.com/commerce/DocumentDelivery/DDEController?Action=srchrtrv&DocNm=SMPM_Connectors_Product_Extension-en&DocType=Data+Sheet&DocLang=English&DocFormat=pdf&PartCntxt=2477330-1"
+		(property "Datasheet" "https://tools.molex.com/pdm_docs/sd/733000020_sd.pdf"
 			(at 68.58 176.53 0)
 			(hide yes)
@@
 			)
 		)
-		(property "Description" "SMPM Connector Plug, Male Pin 50 Ohms Board Edge, Cutout; Surface Mount Solder"
+		(property "Description" "SMPM Connector Plug, Male Pin 50Ohm Board Edge, Cutout; Surface Mount Solder"
 			(at 68.58 185.42 0)
 			(hide yes)
@@
 			)
 		)
-		(pin "SHLD"
+		(pin "2"
 		)
-		(pin "SIG"
+		(pin "1"
 		)
 		(instances
 			(project "oresat1-minusz-end-card"
 				(path "/f7595184-4323-4ed9-b19e-5e32e3c6e76f"
-					(reference "CM2")
+					(reference "J2")
 					(unit 1)
 				)
@@
 			)
 		)
-		(pin "MY-UART-RX" input
-			(at 172.72 80.01 0)
-			(effects
-				(font
-					(size 1.27 1.27)
-				)
-				(justify right)
-			)
-		)
-		(pin "MY-UART-TX" input
-			(at 172.72 77.47 0)
-			(effects
-				(font
-					(size 1.27 1.27)
-				)
-				(justify right)
-			)
-		)
 		(pin "PX-UART-RX" input
 			(at 172.72 57.15 0)
@@
 			(effects
 				(font
-					(size 1.27 1.27)
-				)
-				(justify right)
-			)
-		)
-		(pin "PY-UART-RX" input
-			(at 172.72 64.77 0)
-			(effects
-				(font
-					(size 1.27 1.27)
-				)
-				(justify right)
-			)
-		)
-		(pin "PY-UART-TX" input
-			(at 172.72 62.23 0)
-			(effects
-				(font

Commit message: Routine Push
Parts:
- renumbered J1 to CM1, J2 to CM2, J3 to CM3
Changed lines of the file:
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@@
 		(in_pos_files yes)
 		(dnp no)
-		(property "Reference" "J3"
+		(property "Reference" "CM3"
 			(at 74.93 220.98 0)
 			(show_name no)
@@
 			(project "oresat1-minusz-end-card"
 				(path "/f7595184-4323-4ed9-b19e-5e32e3c6e76f"
-					(reference "J3")
+					(reference "CM3")
 					(unit 1)
 				)
@@
 		(in_pos_files yes)
 		(dnp no)
-		(property "Reference" "J1"
+		(property "Reference" "CM1"
 			(at 73.66 158.75 0)
 			(show_name no)
@@
 			(project "oresat1-minusz-end-card"
 				(path "/f7595184-4323-4ed9-b19e-5e32e3c6e76f"
-					(reference "J1")
+					(reference "CM1")
 					(unit 1)
 				)
@@
 		(in_pos_files yes)
 		(dnp no)
-		(property "Reference" "J2"
+		(property "Reference" "CM2"
 			(at 73.66 189.23 0)
 			(show_name no)
@@
 			(project "oresat1-minusz-end-card"
 				(path "/f7595184-4323-4ed9-b19e-5e32e3c6e76f"
-					(reference "J2")
+					(reference "CM2")
 					(unit 1)
 				)

Commit message: Lots of little polishing, checking rules, updating symbols and footprints, adding README and Makefile
Parts:
- HW1, HW2, HW3, HW4, HW5, HW6: DIS McMaster-Carr -> McMaster Carr
Changed lines of the file:
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@@
 			)
 		)
-		(property "DIS" "McMaster-Carr"
+		(property "DIS" "McMaster Carr"
 			(at 238.76 261.62 0)
 			(hide yes)
@@
 			)
 		)
-		(property "DIS" "McMaster-Carr"
+		(property "DIS" "McMaster Carr"
 			(at 238.76 254 0)
 			(hide yes)
@@
 			)
 		)
-		(property "DIS" "McMaster-Carr"
+		(property "DIS" "McMaster Carr"
 			(at 266.7 261.62 0)
 			(hide yes)
@@
 			)
 		)
-		(property "DIS" "McMaster-Carr"
+		(property "DIS" "McMaster Carr"
 			(at 238.76 246.38 0)
 			(hide yes)
@@
 			)
 		)
-		(property "DIS" "McMaster-Carr"
+		(property "DIS" "McMaster Carr"
 			(at 266.7 246.38 0)
 			(hide yes)
@@
 			)
 		)
-		(property "DIS" "McMaster-Carr"
+		(property "DIS" "McMaster Carr"
 			(at 266.7 254 0)
 			(hide yes)
