File: oresat1-minusz-end-card/oresat1-minusz-end-card.kicad_sch (KiCad schematic)
At the start: 31 parts, among them J1 J-SAMTEC-TFM-120-01-L-D-RA, J2 U.FL-R-SMT-1, J3 M55-7101242R, J5 M55-7101242R

Commit message: V1.4 of the -Z end card. Better ground stitching, cleanup, good to go
Other:
- note added: "All resistors are 0603 1% AEC-Q200 unless marked. All capacitors are 0603 AEC-Q200 Vw >= 16V X5R or better unless marked."
Changed lines of the file:
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@@
 	(title_block
 		(title "OreSat1 -Z End Card")
-		(date "2026-09-25")
+		(date "2026-10-21")
 		(rev "v1.4")
 		(company "Portland State Aerospace Society")
@@
 			)
 			(justify left bottom)
+		)
+	)
+	(text "All resistors are 0603 1% AEC-Q200 unless marked.\nAll capacitors are 0603 AEC-Q200 Vw >= 16V X5R or better unless marked."
+		(exclude_from_sim no)
+		(at 113.03 265.938 0)
+		(effects
+			(font
+				(size 1.27 1.27)
+			)
+			(justify left bottom)
