File: oresat1-minusz-end-card/oresat1-minusz-end-card.kicad_pcb (KiCad board)
At the start: 4 copper layers, 99.8 x 94.6 mm, 92 parts, among them J1 J-SAMTEC-TFM-120-01-L-D-RA, J2 U.FL-R-SMT-1, J3 M55-7101242R, J5 M55-7101242R, Q1 DMP2240UDM, Q2 PMV45EN, Q3 PMV45EN, Q4 PMV45EN, Q5 DMP2240UDM-7, Q6 PMV45EN, Q7 DMP2240UDM-7, U11 MIC842LYC5, U12 MIC842LYC5, U2 MAX7310, U201 TS5A21366, U203 TS5A21366

Commit message: Lots of little polishing, checking rules, updating symbols and footprints, adding README and Makefile
Parts:
- moved D1 0.63 mm to (115.7, 147.3)
- moved R99 0.63 mm to (115.7, 144.7)
Routing:
- net /MAG-SDA: track 56.9 -> 50.7 mm, vias 1 -> 2
- net /MAG-POWER: track 54.3 -> 48.3 mm
- net /MAG-SCL: track 56.3 -> 52.1 mm, vias 1 -> 2
- net /~{SD}: track 157.7 -> 158.8 mm, vias 4 -> 6
- net VPD: track 61.6 -> 60.8 mm
- net /OPD/TURNSTILE_DEPLOY: track 46.1 -> 45.4 mm
- net /OPD/PX_UART_EN: track 25.8 -> 25.2 mm
- net GND: vias 323 -> 325
Other:
- board text added: "DEPLOY"
- board text added: "L1 BAND"
- board text removed: "DNP"

Commit message: Feedback from Pete: add opd_pwr cap, make consistent with +Z end card
Parts:
- added C5: 1u, oresat-passives:0603-C-NOSILK, F.Cu at (135.7, 68.7)
Routing:
- net GND: vias 325 -> 326

Commit message: V1.4 of the -Z end card. Better ground stitching, cleanup, good to go
Parts:
- added TP157: Test-Point, oresat-misc:TestPoint_Pad_D1.0mm, F.Cu at (123.5, 121.4)
- added TP158: Test-Point, oresat-misc:TestPoint_Pad_D1.0mm, F.Cu at (125.6, 79.6)
- added TP159: Test-Point, oresat-misc:TestPoint_Pad_D1.0mm, F.Cu at (128.0, 79.6)
- C205: value 470n -> 1u
- Q1: value DMP2240UDM -> DMP2240UDM-7
- Q2, Q3, Q4, Q6: value PMV45EN -> DMN2053UQ-13
- R39, R40, R45, R46, R52, R53, R54, R55, R56, R57, R58, R59: value 1k -> 100
- R99: value 4.7k -> 1k
- moved R95 0.46 mm to (142.3, 132.8)
Connections:
- U2 pad 10: unconnected-(U2-IO5-Pad10) -> Net-(U2-IO5)
- U2 pad 12: unconnected-(U2-IO7-Pad12) -> Net-(U2-IO7)
Routing:
- net GND: track 8.60 -> 0.00 mm, vias 326 -> 368
- net Net-(U2-IO7): track 0.00 -> 2.55 mm
- net Net-(U2-IO5): track 0.00 -> 2.10 mm
- net Net-(Q5A-G): track 20.2 -> 21.6 mm
- net VBUS: vias 36 -> 34
