File: oresat1-plusz-end-card/oresat1-plusz-end-card.kicad_sch (KiCad schematic)
At the start: 35 parts, among them J1 J-SAMTEC-TFM-120-01-L-D-RA, J2 M55-7101242R, J3 M55-7101242R, J4 M55-7101242R, J5 M55-7101242R, J6 U.FL-R-SMT-1

Commit message: Routine push
Connections:
- net GND: now also CM1.2 (SHLD), CM2.2 (SHLD); no longer CM1.SHLD, CM2.SHLD
- net RF_HELICAL: now also CM1.1 (SIG); no longer CM1.SIG
- net RF_PATCH: now also CM2.1 (SIG); no longer CM2.SIG
- net +Z EC OreSat Power Domain (OPD)/MY-UART-RX: no longer names the net of J2.8 (Pin_8)
- net +Z EC OreSat Power Domain (OPD)/MY-UART-TX: no longer names the net of J2.7 (Pin_7)
- net +Z EC OreSat Power Domain (OPD)/PY-UART-RX: no longer names the net of J4.8 (Pin_8)
- net +Z EC OreSat Power Domain (OPD)/PY-UART-TX: no longer names the net of J4.7 (Pin_7)
- no-connect marks 12 -> 16
Other:
- sheet +Z EC OreSat Power Domain (OPD) ports: added none; removed MY-UART-RX, MY-UART-TX, PY-UART-RX, PY-UART-TX
Changed lines of the file:
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@@
 	(title_block
 		(title "OreSat1 +Z End Card")
-		(date "2026-03-23")
-		(rev "v1.1")
+		(date "2026-09-22")
+		(rev "v1.2")
 		(company "Portland State Aerospace Society")
 	)
@@
 	)
 	(no_connect
+		(at 238.76 177.8)
+	)
+	(no_connect
 		(at 67.31 144.78)
 	)
@@
 	)
 	(no_connect
+		(at 238.76 180.34)
+	)
+	(no_connect
+		(at 334.01 180.34)
+	)
+	(no_connect
+		(at 334.01 177.8)
+	)
+	(no_connect
 		(at 67.31 172.72)
 	)
@@
 	(wire
 		(pts
-			(xy 212.09 177.8) (xy 238.76 177.8)
-		)
-		(stroke
-			(width 0)
-			(type default)
-		)
-	)
-	(wire
-		(pts
 			(xy 63.5 40.64) (xy 63.5 41.91)
 		)
@@
 	(wire
 		(pts
-			(xy 321.31 180.34) (xy 321.31 129.54)
-		)
-		(stroke
-			(width 0)
-			(type default)
-		)
-	)
-	(wire
-		(pts
 			(xy 339.09 195.58) (xy 339.09 198.12)
 		)
@@
 	(wire
 		(pts
-			(xy 209.55 180.34) (xy 209.55 144.78)
-		)
-		(stroke
-			(width 0)
-			(type default)
-		)
-	)
-	(wire
-		(pts
 			(xy 99.06 35.56) (xy 114.3 35.56)
 		)
@@
 	(wire
 		(pts
-			(xy 209.55 180.34) (xy 238.76 180.34)
-		)
-		(stroke
-			(width 0)
-			(type default)
-		)
-	)
-	(wire
-		(pts
 			(xy 68.58 69.85) (xy 90.17 69.85)
 		)
@@
 	(wire
 		(pts
-			(xy 323.85 177.8) (xy 334.01 177.8)
-		)
-		(stroke
-			(width 0)
-			(type default)
-		)
-	)
-	(wire
-		(pts
 			(xy 279.4 134.62) (xy 279.4 177.8)
 		)
@@
 	(wire
 		(pts
-			(xy 200.66 144.78) (xy 209.55 144.78)
-		)
-		(stroke
-			(width 0)
-			(type default)
-		)
-	)
-	(wire
-		(pts
 			(xy 67.31 177.8) (xy 68.58 177.8)
 		)
@@
 	(wire
 		(pts
-			(xy 321.31 180.34) (xy 334.01 180.34)
-		)
-		(stroke
-			(width 0)
-			(type default)
-		)
-	)
-	(wire
-		(pts
 			(xy 99.06 35.56) (xy 99.06 36.83)
 		)
@@
 	(wire
 		(pts
-			(xy 200.66 127) (xy 323.85 127)
-		)
-		(stroke
-			(width 0)
-			(type default)
-		)
-	)
-	(wire
-		(pts
-			(xy 321.31 129.54) (xy 200.66 129.54)
-		)
-		(stroke
-			(width 0)
-			(type default)
-		)
-	)
-	(wire
-		(pts
 			(xy 260.35 45.72) (xy 260.35 48.26)
 		)
@@
 	(wire
 		(pts
-			(xy 212.09 142.24) (xy 212.09 177.8)
-		)
-		(stroke
-			(width 0)
-			(type default)
-		)
-	)
-	(wire
-		(pts
 			(xy 68.58 154.94) (xy 81.28 154.94)
 		)
@@
 	(wire
 		(pts
-			(xy 200.66 142.24) (xy 212.09 142.24)
-		)
-		(stroke
-			(width 0)
-			(type default)
-		)
-	)
-	(wire
-		(pts
 			(xy 334.01 187.96) (xy 334.01 190.5)
 		)
@@
 	(wire
 		(pts
-			(xy 323.85 127) (xy 323.85 177.8)
-		)
-		(stroke
-			(width 0)
-			(type default)
-		)
-	)
-	(wire
-		(pts
 			(xy 68.58 160.02) (xy 68.58 157.48)
 		)
@@
 	)
 	(symbol
+		(lib_name "J-MOLEX-SMPM-73300-002X_1")
 		(lib_id "oresat-connectors:J-MOLEX-SMPM-73300-002X")
 		(at 63.5 35.56 0)
@@
 			)
 		)
-		(property "Datasheet" "https://www.te.com/commerce/DocumentDelivery/DDEController?Action=srchrtrv&DocNm=SMPM_Connectors_Product_Extension-en&DocType=Data+Sheet&DocLang=English&DocFormat=pdf&PartCntxt=2477330-1"
+		(property "Datasheet" "https://tools.molex.com/pdm_docs/sd/733000020_sd.pdf"
 			(at 63.5 26.67 0)
 			(hide yes)
@@
 			)
 		)
-		(property "Description" "SMPM Connector Plug, Male Pin 50 Ohms Board Edge, Cutout; Surface Mount Solder"
+		(property "Description" "SMPM Connector Plug, Male Pin 50Ohm Board Edge, Cutout; Surface Mount Solder"
 			(at 63.5 35.56 0)
 			(hide yes)
@@
 			)
 		)
-		(pin "SHLD"
+		(pin "2"
 		)
-		(pin "SIG"
+		(pin "1"
 		)
 		(instances
@@
 			)
 		)
-		(property "Datasheet" "https://www.te.com/commerce/DocumentDelivery/DDEController?Action=srchrtrv&DocNm=SMPM_Connectors_Product_Extension-en&DocType=Data+Sheet&DocLang=English&DocFormat=pdf&PartCntxt=2477330-1"
+		(property "Datasheet" "https://tools.molex.com/pdm_docs/sd/733000020_sd.pdf"
 			(at 63.5 60.96 0)
 			(hide yes)
@@
 			)
 		)
-		(property "Description" "SMPM Connector Plug, Male Pin 50 Ohms Board Edge, Cutout; Surface Mount Solder"
+		(property "Description" "SMPM Connector Plug, Male Pin 50Ohm Board Edge, Cutout; Surface Mount Solder"
 			(at 63.5 69.85 0)
 			(hide yes)
@@
 			)
 		)
-		(pin "SHLD"
+		(pin "2"
 		)
-		(pin "SIG"
+		(pin "1"
 		)
 		(instances
@@
 			)
 		)
-		(pin "MY-UART-RX" input
-			(at 200.66 144.78 0)
-			(effects
-				(font
-					(size 1.27 1.27)
-				)
-				(justify right)
-			)
-		)
-		(pin "MY-UART-TX" input
-			(at 200.66 142.24 0)
-			(effects
-				(font
-					(size 1.27 1.27)
-				)
-				(justify right)
-			)
-		)
 		(pin "PX-UART-RX" input
 			(at 200.66 137.16 0)
@@
 			(effects
 				(font
-					(size 1.27 1.27)
-				)
-				(justify right)
-			)
-		)
-		(pin "PY-UART-RX" input
-			(at 200.66 129.54 0)
-			(effects
-				(font
-					(size 1.27 1.27)
-				)
-				(justify right)
-			)
-		)
-		(pin "PY-UART-TX" input
-			(at 200.66 127 0)
-			(effects
-				(font

Commit message: Polishing schematic, syncing, polishing layout, added releases folder, updating makefile
Parts:
- HW10, HW11, HW12, HW13, HW14, HW4, HW9: DIS McMaster-Carr -> McMaster Carr
Changed lines of the file:
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@@
 			)
 		)
-		(property "DIS" "McMaster-Carr"
+		(property "DIS" "McMaster Carr"
 			(at 248.92 254 0)
 			(hide yes)
@@
 			)
 		)
-		(property "DIS" "McMaster-Carr"
+		(property "DIS" "McMaster Carr"
 			(at 278.13 238.76 0)
 			(hide yes)
@@
 			)
 		)
-		(property "DIS" "McMaster-Carr"
+		(property "DIS" "McMaster Carr"
 			(at 248.92 238.76 0)
 			(hide yes)
@@
 			)
 		)
-		(property "DIS" "McMaster-Carr"
+		(property "DIS" "McMaster Carr"
 			(at 278.13 246.38 0)
 			(hide yes)
@@
 			)
 		)
-		(property "DIS" "McMaster-Carr"
+		(property "DIS" "McMaster Carr"
 			(at 278.13 231.14 0)
 			(hide yes)
@@
 			)
 		)
-		(property "DIS" "McMaster-Carr"
+		(property "DIS" "McMaster Carr"
 			(at 248.92 231.14 0)
 			(hide yes)
@@
 			)
 		)
-		(property "DIS" "McMaster-Carr"
+		(property "DIS" "McMaster Carr"
 			(at 248.92 246.38 0)
 			(hide yes)
